File: MDCC_1024k.brd (EAGLE design)
At the start: 62.2 x 84 mm, 12 parts, among them IC1 74LS273, IC2 74LS02, IC3 29F040, IC4 29F040

Commit message: Add files via upload
Parts:
- added LOCK: (no value), SparkFun-Passives:SJ_3
Connections:
- new net N$3: IC2.3, LOCK.2
- net DIS: now also LOCK.3; no longer IC2.3
- net GND: now also LOCK.1
Routing:
- net GND: track 238.9 -> 250.9 mm, vias 2 -> 3
- net N$3: track 0.00 -> 4.69 mm
- net CE2: track 40.5 -> 38.3 mm, vias 2 -> 0
Other:
- board text added: "LOCK NO LOCK"
Changed lines of the file:
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@@
 <text x="24.8846" y="69.3996" size="1.6764" layer="29" font="vector" ratio="15" distance="30" rot="SR0" align="center">COMPATIBLE CARTRIDGE</text>
 <text x="13.9446" y="32.4104" size="1.016" layer="26" font="vector" ratio="12" distance="30" rot="SMR270" align="center">https://github.com/msolajic/c64-magic-desk-1024k</text>
+<wire x1="18.415" y1="62.865" x2="19.05" y2="62.865" width="0.4064" layer="30"/>
+<text x="17.1704" y="62.8904" size="0.8128" layer="26" font="vector" ratio="12" distance="30" rot="SMR0" align="center">LOCK     NO LOCK</text>
 </plain>
 <attributes>
@@
 <attribute name="OC_FARNELL" value="176432" x="20.32" y="78.105" size="1.778" layer="27" rot="R90" display="off"/>
 </element>
+<element name="LOCK" library="SparkFun-Passives" package="SJ_3" value="" x="18.415" y="62.865" smashed="yes" rot="MR180">
+<attribute name="VALUE" x="18.3149" y="62.865" size="0.02" layer="28" rot="MR180"/>
+<attribute name="VALUE" x="17.145" y="64.77" size="0.4064" layer="28" rot="MR180"/>
+</element>
 </elements>
 <signals>
@@
 <wire x1="55.8546" y1="59.0804" x2="59.0296" y2="55.9054" width="0.4064" layer="16"/>
 <polygon width="0.4064" layer="1" isolate="0.4064">
-<vertex x="-0.635" y="85.725"/>
+<vertex x="0" y="85.725"/>
 <vertex x="65.405" y="85.725"/>
 <vertex x="65.405" y="9.525"/>
-<vertex x="-0.635" y="9.525"/>
+<vertex x="0" y="9.525"/>
 </polygon>
 <polygon width="0.4064" layer="16" isolate="0.4064">
 <vertex x="66.675" y="86.995"/>
-<vertex x="-1.905" y="86.995"/>
-<vertex x="-1.905" y="9.525"/>
+<vertex x="-1.27" y="86.995"/>
+<vertex x="-1.27" y="9.525"/>
 <vertex x="66.675" y="9.525"/>
 </polygon>
@@
 <wire x1="22.225" y1="74.93" x2="22.225" y2="81.0006" width="0.4064" layer="16"/>
 <wire x1="22.225" y1="81.0006" x2="22.5806" y2="81.3562" width="0.4064" layer="16"/>
+<contactref element="LOCK" pad="1"/>
+<wire x1="17.526" y1="62.865" x2="17.526" y2="63.881" width="0.4064" layer="16"/>
+<wire x1="17.526" y1="63.881" x2="17.78" y2="64.135" width="0.4064" layer="16"/>
+<via x="17.78" y="64.135" extent="1-16" drill="0.6" shape="octagon"/>
+<wire x1="17.78" y1="64.135" x2="12.7" y2="64.135" width="0.4064" layer="1"/>
+<wire x1="12.7" y1="64.135" x2="10.16" y2="61.595" width="0.4064" layer="1"/>
+<wire x1="10.16" y1="61.595" x2="8.255" y2="61.595" width="0.4064" layer="1"/>
+<wire x1="8.255" y1="61.595" x2="8.2296" y2="61.6204" width="0.4064" layer="1"/>
 </signal>
 <signal name="VCC">
@@
 <signal name="DIS">
 <contactref element="U$1" pad="9"/>
-<contactref element="IC2" pad="3"/>
 <contactref element="IC1" pad="19"/>
 <wire x1="25.3846" y1="4.3354" x2="25.3746" y2="8.2804" width="0.4064" layer="1"/>
@@
 <wire x1="20.2946" y1="8.9154" x2="17.7546" y2="11.4554" width="0.4064" layer="1"/>
 <via x="17.7546" y="11.4554" extent="1-16" drill="0.6" shape="octagon"/>
-<wire x1="17.7546" y1="11.4554" x2="17.7546" y2="59.0804" width="0.4064" layer="16"/>
 <wire x1="35.5346" y1="66.7004" x2="35.5346" y2="65.4304" width="0.4064" layer="1"/>
 <wire x1="35.5346" y1="65.4304" x2="34.8996" y2="64.7954" width="0.4064" layer="1"/>
 <wire x1="34.8996" y1="64.7954" x2="19.0246" y2="64.7954" width="0.4064" layer="1"/>
 <via x="19.0246" y="64.7954" extent="1-16" drill="0.6" shape="octagon"/>
-<wire x1="19.0246" y1="64.7954" x2="18.3896" y2="64.7954" width="0.4064" layer="16"/>
-<wire x1="18.3896" y1="64.7954" x2="17.7546" y2="64.1604" width="0.4064" layer="16"/>
-<wire x1="17.7546" y1="64.1604" x2="17.7546" y2="59.0804" width="0.4064" layer="16"/>
+<contactref element="LOCK" pad="3"/>
+<wire x1="17.7546" y1="11.4554" x2="17.7546" y2="56.4896" width="0.4064" layer="16"/>
+<wire x1="17.7546" y1="56.4896" x2="19.05" y2="57.785" width="0.4064" layer="16"/>
+<wire x1="19.304" y1="62.865" x2="19.304" y2="60.579" width="0.4064" layer="16"/>
+<wire x1="19.304" y1="60.579" x2="19.05" y2="60.325" width="0.4064" layer="16"/>
+<wire x1="19.05" y1="60.325" x2="19.05" y2="57.785" width="0.4064" layer="16"/>
+<wire x1="19.304" y1="62.865" x2="19.304" y2="64.516" width="0.4064" layer="16"/>
+<wire x1="19.304" y1="64.516" x2="19.0246" y2="64.7954" width="0.4064" layer="16"/>
 </signal>
 <signal name="ROML">
@@
 <contactref element="IC2" pad="10"/>
 <contactref element="IC4" pad="24"/>
-<wire x1="19.0246" y1="63.5254" x2="19.0246" y2="33.6804" width="0.4064" layer="16"/>
 <wire x1="19.0246" y1="33.6804" x2="20.2946" y2="32.4104" width="0.4064" layer="16"/>
 <wire x1="20.2946" y1="32.4104" x2="22.1996" y2="32.4104" width="0.4064" layer="16"/>
-<via x="19.0246" y="63.5254" extent="1-16" drill="0.6" shape="octagon"/>
-<wire x1="19.0246" y1="63.5254" x2="22.8346" y2="63.5254" width="0.4064" layer="1"/>
-<via x="22.8346" y="63.5254" extent="1-16" drill="0.6" shape="octagon"/>
-<wire x1="22.8346" y1="63.5254" x2="22.8346" y2="66.7004" width="0.4064" layer="16"/>
+<wire x1="22.8346" y1="62.8396" x2="22.8346" y2="66.7004" width="0.4064" layer="16"/>
+<wire x1="22.8346" y1="62.8396" x2="21.59" y2="61.595" width="0.4064" layer="16"/>
+<wire x1="21.59" y1="61.595" x2="21.59" y2="57.785" width="0.4064" layer="16"/>
+<wire x1="21.59" y1="57.785" x2="19.05" y2="55.245" width="0.4064" layer="16"/>
+<wire x1="19.05" y1="55.245" x2="19.05" y2="33.7058" width="0.4064" layer="16"/>
+<wire x1="19.05" y1="33.7058" x2="19.0246" y2="33.6804" width="0.4064" layer="16"/>
 </signal>
 <signal name="PIN1">
@@
 <via x="24.13" y="78.74" extent="1-16" drill="1.524"/>
 </signal>
+<signal name="N$3">
+<contactref element="IC2" pad="3"/>
+<contactref element="LOCK" pad="2"/>
+<wire x1="17.7546" y1="59.0804" x2="17.7546" y2="60.2996" width="0.4064" layer="16"/>
+<wire x1="18.415" y1="62.865" x2="18.415" y2="60.96" width="0.4064" layer="16"/>
+<wire x1="18.415" y1="60.96" x2="17.7546" y2="60.2996" width="0.4064" layer="16"/>
+<wire x1="18.415" y1="62.865" x2="19.05" y2="62.865" width="0.254" layer="16"/>
+</signal>
 </signals>
